File: Routage_3IMACS_gpeC_Gilbert_Frouin.kicad_pcb (KiCad board)
At the start: 2 copper layers, 52 parts, among them J2 Conn_01x02, J3 Conn_01x03, Q1 2N2907, Q10 TIP31, Q11 BD138, Q12 TIP31, Q13 2N2222, Q2 2N2907, Q3 2N2907, Q4 2N2222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

Commit message: etape2
Routing:
- net -12V: track 212.8 -> 218.3 mm
- net GND: track 136.7 -> 140.3 mm
- net +12V: track 90.6 -> 93.2 mm
Other:
- board text added: "Valentin Gilbert - Mathis Frouin Routage amplificateur audio 3IMACS 2020"
Changed lines of the file:
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@@
   (general
     (thickness 1.6)
-    (drawings 4)
-    (tracks 262)
+    (drawings 5)
+    (tracks 272)
     (zones 0)
     (modules 52)
@@
   )
   (setup
-    (last_trace_width 2)
+    (last_trace_width 0.4)
     (user_trace_width 0.4)
     (user_trace_width 0.5)
@@
       (net 2 /JC1))
   )
+  (gr_text "Valentin Gilbert - Mathis Frouin\nRoutage amplificateur audio\n3IMACS 2020" (at 144.653 101.473 90) (layer Margin)
+    (effects (font (size 1.5 1.5) (thickness 0.3)))
+  )
   (gr_line (start 151.148 77.724) (end 151.148 177.724) (layer F.SilkS) (width 0.12))
   (gr_line (start 41.148 177.724) (end 41.148 77.724) (layer F.SilkS) (width 0.12))
@@
   (segment (start 94.701179 154.772179) (end 101.940179 154.772179) (width 1) (layer F.Cu) (net 5))
   (segment (start 89.027 160.274) (end 90.043 160.274) (width 1) (layer B.Cu) (net 5))
-  (segment (start 86.868 158.115) (end 89.027 160.274) (width 1) (layer B.Cu) (net 5))
   (segment (start 91.186 159.131) (end 91.186 158.287358) (width 1) (layer B.Cu) (net 5))
   (segment (start 90.043 160.274) (end 91.186 159.131) (width 1) (layer B.Cu) (net 5))
@@
   (segment (start 87.503 164.090498) (end 89.281 162.312498) (width 2) (layer B.Cu) (net 5))
   (segment (start 87.503 165.434) (end 87.503 164.090498) (width 2) (layer B.Cu) (net 5))
-  (segment (start 89.281 160.528) (end 86.36 157.607) (width 2) (layer B.Cu) (net 5))
   (segment (start 86.36 152.908) (end 89.408 149.86) (width 2) (layer B.Cu) (net 5))
   (segment (start 86.36 157.607) (end 86.36 152.908) (width 2) (layer B.Cu) (net 5))
@@
   (segment (start 95.553002 149.86) (end 99.949 145.464002) (width 2) (layer B.Cu) (net 5))
   (segment (start 90.17 149.86) (end 89.408 149.86) (width 1) (layer B.Cu) (net 5))
+  (segment (start 88.646 159.893) (end 89.580358 159.893) (width 0.5) (layer B.Cu) (net 5))
+  (segment (start 88.646 159.893) (end 89.027 160.274) (width 1) (layer B.Cu) (net 5))
+  (segment (start 86.868 158.115) (end 88.646 159.893) (width 1) (layer B.Cu) (net 5))
+  (segment (start 90.043 159.512) (end 90.424 159.131) (width 0.5) (layer B.Cu) (net 5))
+  (segment (start 88.265 159.512) (end 90.043 159.512) (width 0.5) (layer B.Cu) (net 5))
+  (segment (start 89.281 160.528) (end 88.265 159.512) (width 2) (layer B.Cu) (net 5))
+  (segment (start 88.265 159.512) (end 86.36 157.607) (width 2) (layer B.Cu) (net 5))
+  (segment (start 89.580358 159.893) (end 90.424 159.131) (width 0.5) (layer B.Cu) (net 5))
+  (segment (start 90.424 159.131) (end 91.186 158.287358) (width 0.5) (layer B.Cu) (net 5))
   (segment (start 94.488 164.45337) (end 94.488 163.322) (width 1) (layer B.Cu) (net 6))
   (segment (start 94.488 165.399) (end 94.488 164.45337) (width 1) (layer B.Cu) (net 6))
@@
   (segment (start 114.708 170.842) (end 110.998 174.552) (width 1) (layer B.Cu) (net 7))
   (segment (start 126.238 113.284) (end 128.778 115.824) (width 2) (layer B.Cu) (net 7))
-  (segment (start 131.25149 115.824) (end 133.604 118.17651) (width 2) (layer B.Cu) (net 7))
-  (segment (start 128.778 115.824) (end 131.25149 115.824) (width 2) (layer B.Cu) (net 7))
   (segment (start 142.875 127.254) (end 137.033 121.412) (width 2) (layer B.Cu) (net 7))
   (segment (start 141.63 164.084) (end 142.875 162.839) (width 2) (layer B.Cu) (net 7))
   (segment (start 138.43 164.084) (end 141.63 164.084) (width 2) (layer B.Cu) (net 7))
   (segment (start 142.875 162.839) (end 142.875 127.254) (width 2) (layer B.Cu) (net 7))
-  (segment (start 133.604 118.17651) (end 137.033 121.412) (width 1) (layer B.Cu) (net 7))
+  (segment (start 133.604 120.65) (end 126.238 113.284) (width 2) (layer B.Cu) (net 7))
+  (segment (start 137.033 121.412) (end 136.271 120.65) (width 2) (layer B.Cu) (net 7))
+  (segment (start 136.271 120.65) (end 133.604 120.65) (width 2) (layer B.Cu) (net 7))
   (segment (start 44.323 136.144) (end 43.688 135.509) (width 1) (layer F.Cu) (net 8))
   (segment (start 121.839 107.107) (end 121.412 106.68) (width 1) (layer F.Cu) (net 8))
@@
   (segment (start 108.712 157.988) (end 108.966 158.242) (width 1) (layer B.Cu) (net 8))
   (segment (start 105.664 157.988) (end 108.712 157.988) (width 1) (layer B.Cu) (net 8))
-  (segment (start 110.766 158.242) (end 108.966 158.242) (width 1) (layer B.Cu) (net 8))
-  (segment (start 137.668 131.34) (end 110.766 158.242) (width 1) (layer B.Cu) (net 8))
-  (segment (start 121.839 118.237) (end 128.397 118.237) (width 1) (layer B.Cu) (net 8))
-  (segment (start 128.397 118.237) (end 133.096 122.936) (width 1) (layer B.Cu) (net 8))
-  (segment (start 133.096 122.936) (end 135.128 122.936) (width 1) (layer B.Cu) (net 8))
-  (segment (start 137.668 125.476) (end 137.668 131.34) (width 1) (layer B.Cu) (net 8))
-  (segment (start 135.128 122.936) (end 137.668 125.476) (width 1) (layer B.Cu) (net 8))
   (segment (start 106.934 110.998) (end 111.252 106.68) (width 2) (layer B.Cu) (net 8))
   (segment (start 102.362 110.998) (end 106.934 110.998) (width 2) (layer B.Cu) (net 8))
   (segment (start 111.252 106.68) (end 121.412 106.68) (width 2) (layer B.Cu) (net 8))
+  (segment (start 121.839 118.237) (end 124.079 118.237) (width 1) (layer B.Cu) (net 8))
+  (segment (start 123.571 118.745) (end 124.079 118.237) (width 0.4) (layer B.Cu) (net 8))
+  (segment (start 124.079 118.237) (end 122.809 116.967) (width 0.4) (layer B.Cu) (net 8))
+  (segment (start 110.766 158.242) (end 108.966 158.242) (width 1) (layer B.Cu) (net 8))
+  (segment (start 137.668 131.34) (end 110.766 158.242) (width 1) (layer B.Cu) (net 8))
+  (segment (start 127 118.237) (end 131.699 122.936) (width 1) (layer B.Cu) (net 8))
+  (segment (start 124.079 118.237) (end 127 118.237) (width 1) (layer B.Cu) (net 8))
+  (segment (start 135.128 122.936) (end 137.668 125.476) (width 1) (layer B.Cu) (net 8))
+  (segment (start 131.699 122.936) (end 135.128 122.936) (width 1) (layer B.Cu) (net 8))
+  (segment (start 137.668 125.476) (end 137.668 131.34) (width 1) (layer B.Cu) (net 8))
   (segment (start 114.106 165.862) (end 114.708 166.464) (width 1) (layer B.Cu) (net 9))
   (segment (start 108.966 165.862) (end 114.106 165.862) (width 1) (layer B.Cu) (net 9))

Commit message: Etape3
Parts:
- moved R8 14.3 mm to (66.4, 113.8), turned to 0 degrees
- moved R6 4.96 mm to (58.8, 117.6)
- moved Q4 4.83 mm to (65.7, 121.9)
- moved Q5 4.83 mm to (74.4, 121.9)
- moved C2 4.83 mm to (71.6, 129.3)
- moved R2 3.05 mm to (77.9, 135.8)
- moved R3 2.40 mm to (58.2, 135.9)
- moved Q11 1.52 mm to (83.6, 130.3)
- moved HS2 0.89 mm to (98.2, 146.8)
- moved R16 0.89 mm to (105.7, 158.9)
Routing:
- net -12V: track 218.3 -> 5.73 mm, vias 2 -> 0
- net Net-(C2-Pad2): track 79.2 -> 50.0 mm
- net Net-(C2-Pad1): track 48.8 -> 72.2 mm
- net GND: track 140.3 -> 122.8 mm
- net +12V: track 93.2 -> 104.6 mm, vias 0 -> 2
- net Net-(Q2-Pad2): track 22.4 -> 32.2 mm
- net Net-(Q5-Pad1): track 17.6 -> 23.3 mm
- net Net-(Q2-Pad3): track 6.03 -> 11.4 mm
- net Net-(D1-Pad2): track 70.3 -> 74.8 mm, vias 0 -> 2
- net Net-(Q11-Pad2): track 28.8 -> 25.9 mm
- net Net-(Q11-Pad1): track 25.5 -> 24.0 mm
- net Net-(C3-Pad1): track 16.9 -> 16.0 mm
Other:
- board text added: "BOTTOM"
- board text added: "TOP"
- board text added: "Valentin Gilbert - Mathis Frouin Routage amplificateur audio 3 IMACS 2020"
- board text removed: "Valentin Gilbert - Mathis Frouin Routage amplificateur audio 3IMACS 2020"

Commit message: Etape4
Parts:
- moved Q10 0.38 mm to (102.0, 105.9)
- moved Q12 0.38 mm to (94.9, 143.4)
Routing:
- net GND: track 122.8 -> 183.4 mm, vias 0 -> 2
- net Net-(Q5-Pad1): track 23.3 -> 17.4 mm
Other:
- board text removed: "TOP"
Changed lines of the file:
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@@
   (general
     (thickness 1.6)
-    (drawings 7)
-    (tracks 230)
+    (drawings 6)
+    (tracks 253)
     (zones 0)
     (modules 52)
@@
   )
   (setup
-    (last_trace_width 1)
+    (last_trace_width 2)
     (user_trace_width 0.4)
     (user_trace_width 0.5)
@@
   )
   (module Lib3imacsCorrige:TO-220-3_Vertical (layer F.Cu)
-    (at 102.362 105.918 270)
+    (at 101.981 105.918 270)
     (descr "TO-220-3, Vertical, RM 2.54mm, see https://www.vishay.com/docs/66542/to-220-1.pdf")
     (tags "TO-220-3 Vertical RM 2.54mm")
@@
   )
   (module Lib3imacsCorrige:TO-220-3_Vertical (layer F.Cu)
-    (at 94.869 143.764)
+    (at 94.869 143.383)
     (descr "TO-220-3, Vertical, RM 2.54mm, see https://www.vishay.com/docs/66542/to-220-1.pdf")
     (tags "TO-220-3 Vertical RM 2.54mm")
@@
       (net 2 /JC1))
   )
-  (gr_text "Valentin Gilbert - Mathis Frouin\nRoutage amplificateur audio\n3 IMACS 2020" (at 145.161 103.632 90) (layer F.Cu)
-    (effects (font (size 1.5 1.5) (thickness 0.3)))
-  )
-  (gr_text TOP (at 46.228 87.757) (layer F.Cu)
-    (effects (font (size 3 3) (thickness 0.5)))
+  (gr_text "Valentin Gilbert - Mathis Frouin\nRoutage amplificateur audio\n3 IMACS 2020" (at 145.161 103.632 90) (layer B.Cu)
+    (effects (font (size 1.5 1.5) (thickness 0.3)) (justify mirror))
   )
   (gr_text BOTTOM (at 135.636 175.133) (layer B.Cu)
@@
   (segment (start 76.962 133.223) (end 77.851 134.112) (width 1) (layer B.Cu) (net 4))
   (segment (start 72.009 133.223) (end 72.009 143.256) (width 1) (layer F.Cu) (net 4))
-  (via (at 118.491 152.146) (size 1.9) (drill 0.6) (layers F.Cu B.Cu) (net 9))
-  (via (at 121.666 161.417) (size 1.9) (drill 0.6) (layers F.Cu B.Cu) (net 8))
   (segment (start 66.468 100.584) (end 66.468 103.204) (width 2) (layer B.Cu) (net 5))
-  (segment (start 99.949 145.464002) (end 99.949 143.764) (width 2) (layer B.Cu) (net 5))
   (segment (start 66.468 100.584) (end 66.468 101.927502) (width 2) (layer B.Cu) (net 5))
   (segment (start 66.468 101.927502) (end 66.421 101.974502) (width 2) (layer B.Cu) (net 5))
+  (segment (start 99.949 143.383) (end 99.949 145.288) (width 2) (layer B.Cu) (net 5))
   (segment (start 94.488 164.45337) (end 94.488 163.322) (width 1) (layer B.Cu) (net 6))
   (segment (start 94.488 165.399) (end 94.488 164.45337) (width 1) (layer B.Cu) (net 6))
@@
   (segment (start 76.708 161.798) (end 74.549 159.639) (width 1) (layer B.Cu) (net 7))
   (segment (start 75.136999 173.529001) (end 76.708 171.958) (width 1) (layer B.Cu) (net 7))
-  (segment (start 59.563 82.679) (end 61.978 80.264) (width 1) (layer B.Cu) (net 7))
-  (segment (start 59.563 83.439) (end 59.563 82.679) (width 1) (layer B.Cu) (net 7))
   (segment (start 61.978 80.264) (end 67.183 80.264) (width 1) (layer B.Cu) (net 7))
-  (segment (start 70.993 84.074) (end 70.993 106.299) (width 1) (layer B.Cu) (net 7))
-  (segment (start 67.183 80.264) (end 70.993 84.074) (width 1) (layer B.Cu) (net 7))
   (segment (start 121.158 174.498) (end 119.842 174.498) (width 1) (layer B.Cu) (net 7))
   (segment (start 135.128 120.65) (end 127.762 113.284) (width 2) (layer B.Cu) (net 7))
@@
   (segment (start 142.875 162.839) (end 142.875 127.254) (width 2) (layer B.Cu) (net 7))
   (segment (start 142.875 127.254) (end 136.271 120.65) (width 2) (layer B.Cu) (net 7))
+  (segment (start 70.993 84.074) (end 70.993 85.09) (width 1) (layer B.Cu) (net 7))
+  (segment (start 88.392 85.09) (end 94.361 91.059) (width 2) (layer B.Cu) (net 7))
+  (segment (start 70.993 85.09) (end 70.993 84.963) (width 1) (layer B.Cu) (net 7))
+  (segment (start 70.993 87.757) (end 71.12 87.757) (width 2) (layer B.Cu) (net 7))
+  (segment (start 70.993 106.299) (end 70.993 87.757) (width 2) (layer B.Cu) (net 7))
+  (segment (start 70.993 85.09) (end 73.787 85.09) (width 2) (layer B.Cu) (net 7))
+  (segment (start 71.12 87.757) (end 73.787 85.09) (width 2) (layer B.Cu) (net 7))
+  (segment (start 70.993 87.757) (end 70.993 84.963) (width 2) (layer B.Cu) (net 7))
+  (segment (start 73.787 85.09) (end 88.392 85.09) (width 2) (layer B.Cu) (net 7))
+  (segment (start 70.993 84.455) (end 67.818 81.28) (width 2) (layer B.Cu) (net 7))
+  (segment (start 70.993 84.963) (end 70.993 84.455) (width 2) (layer B.Cu) (net 7))
+  (segment (start 67.183 80.264) (end 67.818 81.28) (width 1) (layer B.Cu) (net 7))
+  (segment (start 67.818 81.28) (end 70.993 84.074) (width 1) (layer B.Cu) (net 7))
+  (segment (start 115.038 83.844) (end 115.038 83.971) (width 2) (layer B.Cu) (net 7))
+  (segment (start 116.078 82.804) (end 115.038 83.844) (width 2) (layer B.Cu) (net 7))
+  (segment (start 115.038 83.971) (end 112.649 86.36) (width 2) (layer B.Cu) (net 7))
+  (segment (start 112.649 86.36) (end 100.076 86.36) (width 2) (layer B.Cu) (net 7))
+  (segment (start 94.361 91.059) (end 94.361 91.059) (width 2) (layer B.Cu) (net 7))
+  (via (at 94.361 91.059) (size 1.9) (drill 0.6) (layers F.Cu B.Cu) (net 7))
+  (segment (start 100.076 86.36) (end 100.076 86.36) (width 2) (layer B.Cu) (net 7))
+  (via (at 99.314 85.979) (size 1.9) (drill 0.6) (layers F.Cu B.Cu) (net 7))
+  (segment (start 99.695 85.979) (end 100.076 86.36) (width 2) (layer B.Cu) (net 7))
+  (segment (start 99.314 85.979) (end 99.695 85.979) (width 2) (layer B.Cu) (net 7))
+  (segment (start 94.361 90.932) (end 99.314 85.979) (width 2) (layer F.Cu) (net 7))
+  (segment (start 94.361 91.059) (end 94.361 90.932) (width 2) (layer F.Cu) (net 7))
+  (segment (start 59.563 82.679) (end 61.5325 80.7095) (width 2) (layer B.Cu) (net 7))
+  (segment (start 59.563 83.439) (end 59.563 82.679) (width 2) (layer B.Cu) (net 7))
+  (segment (start 61.5325 80.7095) (end 61.978 80.264) (width 1) (layer B.Cu) (net 7))
+  (via (at 121.666 161.417) (size 1.9) (drill 0.6) (layers F.Cu B.Cu) (net 8))
   (segment (start 44.323 136.144) (end 43.688 135.509) (width 1) (layer F.Cu) (net 8))
   (segment (start 121.839 107.107) (end 121.412 106.68) (width 1) (layer F.Cu) (net 8))
@@
   (segment (start 108.712 157.988) (end 108.966 158.242) (width 1) (layer B.Cu) (net 8))
   (segment (start 106.934 110.998) (end 111.252 106.68) (width 2) (layer B.Cu) (net 8))
-  (segment (start 102.362 110.998) (end 106.934 110.998) (width 2) (layer B.Cu) (net 8))
   (segment (start 111.252 106.68) (end 121.412 106.68) (width 2) (layer B.Cu) (net 8))
   (segment (start 121.839 118.237) (end 124.079 118.237) (width 1) (layer B.Cu) (net 8))
@@
   (segment (start 118.618 159.512) (end 118.645999 159.539999) (width 1) (layer B.Cu) (net 8))
   (segment (start 112.036 159.512) (end 118.618 159.512) (width 1) (layer B.Cu) (net 8))
+  (segment (start 101.981 110.998) (end 106.934 110.998) (width 2) (layer B.Cu) (net 8))
+  (via (at 118.491 152.146) (size 1.9) (drill 0.6) (layers F.Cu B.Cu) (net 9))
   (segment (start 114.106 165.862) (end 114.708 166.464) (width 1) (layer B.Cu) (net 9))
   (segment (start 108.966 165.862) (end 114.106 165.862) (width 1) (layer B.Cu) (net 9))
@@
   (segment (start 71.552 121.72) (end 73.022 123.19) (width 1) (layer B.Cu) (net 17))
   (segment (start 65.759 121.72) (end 71.552 121.72) (width 1) (layer B.Cu) (net 17))
-  (segment (start 70.404 117.602) (end 74.522 121.72) (width 1) (layer B.Cu) (net 18))
   (segment (start 73.772001 120.970001) (end 74.522 121.72) (width 1) (layer B.Cu) (net 18))
   (segment (start 71.353999 118.551999) (end 73.772001 120.970001) (width 1) (layer B.Cu) (net 18))
@@
   (segment (start 105.791 103.632) (end 99.187 97.028) (width 1) (layer B.Cu) (net 24))
   (segment (start 105.791 107.061) (end 105.791 103.632) (width 1) (layer B.Cu) (net 24))
-  (segment (start 102.362 108.458) (end 104.394 108.458) (width 1) (layer B.Cu) (net 24))
   (segment (start 104.394 108.458) (end 105.791 107.061) (width 1) (layer B.Cu) (net 24))
-  (segment (start 97.649998 108.458) (end 102.362 108.458) (width 1) (layer B.Cu) (net 24))
   (segment (start 95.758 107.696) (end 96.52 108.458) (width 1) (layer B.Cu) (net 24))
   (segment (start 96.52 108.458) (end 97.649998 108.458) (width 1) (layer B.Cu) (net 24))
-  (segment (start 96.012 99.568) (end 102.362 105.918) (width 1) (layer B.Cu) (net 25))
-  (segment (start 95.25 99.568) (end 96.012 99.568) (width 1) (layer B.Cu) (net 25))
+  (segment (start 97.649998 108.458) (end 101.981 108.458) (width 1) (layer B.Cu) (net 24))
+  (segment (start 101.981 108.458) (end 104.394 108.458) (width 1) (layer B.Cu) (net 24))
+  (segment (start 95.631 99.568) (end 101.981 105.918) (width 1) (layer B.Cu) (net 25))
+  (segment (start 95.25 99.568) (end 95.631 99.568) (width 1) (layer B.Cu) (net 25))
   (segment (start 91.694 130.302) (end 94.742 133.35) (width 1) (layer B.Cu) (net 26))
   (segment (start 97.409 136.017) (end 94.742 133.35) (width 1) (layer B.Cu) (net 26))
-  (segment (start 97.409 143.764) (end 97.409 136.017) (width 1) (layer B.Cu) (net 26))
   (segment (start 83.566 130.302) (end 91.694 130.302) (width 1) (layer B.Cu) (net 26))
+  (segment (start 97.409 136.017) (end 97.409 143.383) (width 1) (layer B.Cu) (net 26))
   (segment (start 82.293208 127.762) (end 83.566 127.762) (width 1) (layer B.Cu) (net 27))
   (segment (start 80.772 133.35) (end 80.772 129.283208) (width 1) (layer B.Cu) (net 27))
-  (segment (start 91.186 143.764) (end 80.772 133.35) (width 1) (layer B.Cu) (net 27))
   (segment (start 80.772 129.283208) (end 82.293208 127.762) (width 1) (layer B.Cu) (net 27))
-  (segment (start 94.869 143.764) (end 91.186 143.764) (width 1) (layer B.Cu) (net 27))
+  (segment (start 90.805 143.383) (end 80.772 133.35) (width 1) (layer B.Cu) (net 27))
+  (segment (start 94.869 143.383) (end 90.805 143.383) (width 1) (layer B.Cu) (net 27))
   (segment (start 76.454 113.792) (end 82.804 113.792) (width 1) (layer B.Cu) (net 28))
   (segment (start 73.533 106.299) (end 76.073 106.299) (width 1) (layer B.Cu) (net 29))
